Commit message: Change lidar's visualization

File: urdf/lidar_m10_p.urdf.xacro (robot description, xacro)
@@ -9,5 +9,5 @@
     <link name="${prefix}_base_link">
       <collision>
-        <origin xyz="0 0 0" rpy="0 0 0"/>
+        <origin xyz="0 0 0.1" rpy="0 0 0"/>
         <geometry>
          <mesh filename="package://robotnik_sensors/meshes/lidar_m10_p.STL"/>
@@ -15,5 +15,5 @@
       </collision>
       <visual>
-        <origin xyz="0 0 0" rpy="0 0 0"/>
+        <origin xyz="0 0 0.1" rpy="0 0 0"/>
         <geometry>
             <mesh filename="package://robotnik_sensors/meshes/lidar_m10_p.STL" />
@@ -35,20 +35,8 @@
     <link name="${prefix}_link">
     </link>
-    <!-- Hokuyo sensor for simulation -->
-    <xacro:sensor_lidar_m10_p_gazebo/>
-  </xacro:macro>
-  <xacro:macro name="sensor_lidar_m10_p_gazebo">
     <gazebo reference="${prefix}_link">
-      <!--<xacro:if value="${gpu}">
-        <xacro:property name="ray_type" value="gpu_ray" />
-        <xacro:property name="plugin_lib" value="libgazebo_ros_gpu_laser.so" />
-      </xacro:if>
-      <xacro:unless value="${gpu}">
-        <xacro:property name="ray_type" value="ray" />
-        <xacro:property name="plugin_lib" value="libgazebo_ros_laser.so" />
-      </xacro:unless>-->
       <sensor type="gpu_lidar" name="${prefix}_sensor">
-        <pose>0 0 0 0 0 0</pose>
-        <visualize>false</visualize>
+      <pose>0 0 0.1 0 0 0</pose>
+        <visualize>true</visualize>
         <update_rate>12</update_rate>
         <ray>
@@ -72,9 +60,4 @@
           </noise>
         </ray>
-        <!--<plugin name="${prefix}_controller" filename="${plugin_lib}">
-          <topicName>${prefix_topic}/scan</topicName>
-          <frameName>/${prefix}_link</frameName>
-          <ignoreTfPrefix>1</ignoreTfPrefix>
-        </plugin>-->
       </sensor>
     </gazebo>

Commit message: Correct sensor tag

File: urdf/lidar_m10_p.urdf.xacro (robot description, xacro)
@@ -1,13 +1,13 @@
 <?xml version="1.0"?>
 <robot xmlns:xacro="http://wiki.ros.org/xacro">
-  <xacro:macro name="sensor_lidar_m10_p" params="prefix parent prefix_topic:='front_laser' *origin min_angle:=3.14159 max_angle:=-3.14159 gpu:=^|false include_inertial:=^|true">
-    <joint name="${prefix}_base_joint" type="fixed">
+  <xacro:macro name="sensor_lidar_m10_p" params="id prefix prefix_laser parent *origin min_angle:=3.14159 max_angle:=-3.14159 include_inertial:=^|true">
+    <joint name="${prefix_laser}_base_joint" type="fixed">
       <xacro:insert_block name="origin" />
       <parent link="${parent}"/>
-      <child link="${prefix}_base_link"/>
+      <child link="${prefix_laser}_base_link"/>
     </joint>
-    <link name="${prefix}_base_link">
+    <link name="${prefix_laser}_base_link">
       <collision>
-        <origin xyz="0 0 0.1" rpy="0 0 0"/>
+        <origin xyz="0 0 0.01" rpy="0 0 0"/>
         <geometry>
          <mesh filename="package://robotnik_sensors/meshes/lidar_m10_p.STL"/>
@@ -15,5 +15,5 @@
       </collision>
       <visual>
-        <origin xyz="0 0 0.1" rpy="0 0 0"/>
+        <origin xyz="0 0 0.01" rpy="0 0 0"/>
         <geometry>
             <mesh filename="package://robotnik_sensors/meshes/lidar_m10_p.STL" />
@@ -28,14 +28,14 @@
       </xacro:if>
     </link>
-    <joint name="${prefix}_joint" type="fixed">
-      <origin xyz="0 0 0.02305" rpy="0 0 0"/>
-      <parent link="${prefix}_base_link"/>
-      <child link="${prefix}_link"/>
+    <joint name="${prefix_laser}_joint" type="fixed">
+      <!-- <origin xyz="0 0 0.02305" rpy="0 0 0"/> -->
+      <origin xyz="0.05 0.05 0.05" rpy="0 0 0"/>
+      <parent link="${prefix_laser}_base_link"/>
+      <child link="${prefix_laser}_link"/>
     </joint>
-    <link name="${prefix}_link">
+    <link name="${prefix_laser}_link">
     </link>
-    <gazebo reference="${prefix}_link">
-      <sensor type="gpu_lidar" name="${prefix}_sensor">
-      <pose>0 0 0.1 0 0 0</pose>
+    <gazebo reference="${prefix_laser}_link">
+      <sensor type="gpu_lidar" name="${prefix_laser}_sensor">
         <visualize>true</visualize>
         <update_rate>12</update_rate>
@@ -60,4 +60,6 @@
           </noise>
         </ray>
+        <gz_frame_id>${prefix}${id}/${prefix_laser}_link</gz_frame_id>
+        <topic>scan_${id}</topic>
       </sensor>
     </gazebo>

Commit message: Correct limit angles

File: urdf/lidar_m10_p.urdf.xacro (robot description, xacro)
@@ -1,5 +1,5 @@
 <?xml version="1.0"?>
 <robot xmlns:xacro="http://wiki.ros.org/xacro">
-  <xacro:macro name="sensor_lidar_m10_p" params="id prefix prefix_laser parent *origin min_angle:=3.14159 max_angle:=-3.14159 include_inertial:=^|true">
+  <xacro:macro name="sensor_lidar_m10_p" params="id prefix prefix_laser parent *origin min_angle:=-3.14159 max_angle:=3.14159 include_inertial:=^|true">
     <joint name="${prefix_laser}_base_joint" type="fixed">
       <xacro:insert_block name="origin" />
