Commit message: Change pkg structure

File: urdf/2d_lidar/hokuyo_urg04lx.urdf.xacro (robot description, xacro)
@@ -2,17 +2,5 @@
 <robot name="sensor_hokuyo_urg04lx" xmlns:xacro="http://wiki.ros.org/xacro">
   <xacro:include filename="$(find robotnik_sensors)/urdf/2d_lidar/lidar_2d_plugin.urdf.xacro" />
-  <xacro:macro name="sensor_hokuyo_urg04lx"
-               params="frame_prefix
-                       parent
-                       *origin
-                       gazebo_classic:=false
-                       gazebo_ignition:=false
-                       node_name:=hokuyo_urg04lx
-                       node_namespace:=${None}
-                       topic_prefix:=~/">
-    <!-- node_namespace is used from node_name if not set -->
-    <xacro:if value="${node_namespace == None}">
-      <xacro:property name="node_namespace" value="${node_name}"/>
-    </xacro:if>
+  <xacro:macro name="sensor_hokuyo_urg04lx" params="id frame_prefix name_prefix parent *origin">
     <joint name="${frame_prefix}base_joint" type="fixed">
       <xacro:insert_block name="origin" />
@@ -42,13 +30,11 @@
     <!-- Hokuyo sensor for simulation -->
     <xacro:lidar_2d_plugin
-      node_namespace="${node_namespace}"
-      node_name="${node_name}"
-      gazebo_classic="${gazebo_classic}"
-      gazebo_ignition="${gazebo_ignition}"
+      id="${id}"
+      name_prefix="${name_prefix}"
       min_range="0.06"
       max_range="4.0"
       min_angle="-2.0943"
       max_angle="2.0943"
-      frame_link="${frame_prefix}link"
+      frame_prefix="${frame_prefix}"
       rate="10"
       resolution="0.004359297"

File: urdf/imu/pixhawk.urdf.xacro (robot description, xacro)
@@ -2,13 +2,5 @@
 <robot name="sensor_pixhawk" xmlns:xacro="http://wiki.ros.org/xacro">
   <xacro:include filename="$(find robotnik_sensors)/urdf/imu/imu_plugin.urdf.xacro" />
-  <xacro:macro name="sensor_pixhawk"
-               params="frame_prefix
-                       parent
-                       *origin
-                       gazebo_classic:=false
-                       gazebo_ignition:=false
-                       node_name:=imu
-                       node_namespace:=${None}
-                       topic_prefix:=~/">
+  <xacro:macro name="sensor_pixhawk" params="id frame_prefix name_prefix parent *origin">
     <joint name="${frame_prefix}base_joint" type="fixed">
       <xacro:insert_block name="origin"/>
@@ -46,9 +38,5 @@
     <link name="${frame_prefix}link" />
     <xacro:imu_plugin
-      node_namespace="${node_namespace}"
-      node_name="${node_name}"
-      gazebo_classic="${gazebo_classic}"
-      gazebo_ignition="${gazebo_ignition}"
-      frame_link="${frame_prefix}link"
+      frame_prefix="${frame_prefix}"
       rate="200.0"
     >
