Commit message: Change of camera & gps sensors

File: urdf/camera/axis_m5013.urdf.xacro (robot description, xacro)
@@ -8,13 +8,5 @@
   <xacro:property name="PI" value="3.14159265359"/>
   <xacro:arg name="axis_m5013_controllers_params_file" default=""/> <!-- $(find robotnik_sensors_gazebo)/config/camera/axis_m5013.yaml -->
-  <xacro:macro name="sensor_axis_m5013"
-               params="frame_prefix
-                       parent
-                       *origin
-                       gazebo_classic:=false
-                       gazebo_ignition:=false
-                       node_name:=axis_m5013
-                       node_namespace:=${None}
-                       topic_prefix:=~/">
+  <xacro:macro name="sensor_axis_m5013" params="id frame_prefix name_prefix parent *origin">
     <joint name="${frame_prefix}base_joint" type="fixed">
       <axis xyz="0 1 0"/>
@@ -46,12 +38,12 @@
       </collision>
     </link>
-    <joint name="${frame_prefix}pan_joint" type="revolute">
-      <axis xyz="1 0 0"/>
+    <joint name="${frame_prefix}pan_joint" type="fixed">
+      <!-- <axis xyz="1 0 0"/> -->
       <origin xyz="0.04 0.0 0.0" rpy="0 0 0"/>
       <!-- check the displacement -->
       <parent link="${frame_prefix}base_link"/>
       <child link="${frame_prefix}pan_link"/>
-      <limit effort="${ptz_joint_effort_limit}" velocity="${ptz_joint_velocity_limit}" lower="-3.1416" upper="3.1416"/>
-      <joint_properties damping="${ptz_joint_damping}" friction="{ptz_joint_friction}"/>
+      <!-- <limit effort="${ptz_joint_effort_limit}" velocity="${ptz_joint_velocity_limit}" lower="-3.1416" upper="3.1416"/>
+      <joint_properties damping="${ptz_joint_damping}" friction="{ptz_joint_friction}"/> -->
     </joint>
     <link name="${frame_prefix}pan_link">
@@ -62,11 +54,11 @@
       </inertial>
     </link>
-    <joint name="${frame_prefix}tilt_joint" type="revolute">
-      <axis xyz="0 -1 0"/>
+    <joint name="${frame_prefix}tilt_joint" type="fixed">
+      <!-- <axis xyz="0 -1 0"/> -->
       <origin xyz="0.0 0.0 0.0" rpy="0 ${-PI/2} 0"/>
       <parent link="${frame_prefix}pan_link"/>
       <child link="${frame_prefix}tilt_link"/>
-      <limit effort="${ptz_joint_effort_limit}" velocity="${ptz_joint_velocity_limit}" lower="-1.5708" upper="1.5708"/>
-      <joint_properties damping="${ptz_joint_damping}" friction="{ptz_joint_friction}"/>
+      <!-- <limit effort="${ptz_joint_effort_limit}" velocity="${ptz_joint_velocity_limit}" lower="-1.5708" upper="1.5708"/>
+      <joint_properties damping="${ptz_joint_damping}" friction="{ptz_joint_friction}"/> -->
     </joint>
     <link name="${frame_prefix}tilt_link">
@@ -107,11 +99,6 @@
     <!-- Axis sensor for simulation -->
     <xacro:camera_plugin
-      node_namespace="${node_namespace}"
-      node_name="${node_name}_color"
-      topic_prefix="${topic_prefix}_color"
-      gazebo_classic="${gazebo_classic}"
-      gazebo_ignition="${gazebo_ignition}"
-      optical_frame="${frame_prefix}color_optical_frame"
-      reference_frame="${frame_prefix}color_frame"
+      frame_prefix="${frame_prefix}"
+      name_prefix="${name_prefix}"
       horizontal_fov="45"
       vertical_fov="32"

File: urdf/camera/camera_plugin.urdf.xacro (robot description, xacro)
@@ -2,11 +2,6 @@
 <robot name="camera_plugin" xmlns:xacro="http://wiki.ros.org/xacro">
   <xacro:macro name="camera_plugin" params="
-            node_namespace
-            node_name
-            topic_prefix
-            gazebo_classic
-            gazebo_ignition
-            optical_frame
-            reference_frame
+            frame_prefix
+            name_prefix
             horizontal_fov
             vertical_fov
@@ -17,42 +12,8 @@
             rate
             ">
-    <xacro:if value="${gazebo_classic}">
-      <gazebo reference="${reference_frame}">
-        <sensor name="${node_name}" type="camera">
-          <camera name="${node_name}">
-            <horizontal_fov>${radians(horizontal_fov)}</horizontal_fov>
-            <vertical_fov>${radians(float(vertical_fov))}</vertical_fov>
-            <image>
-              <width>${video_width}</width>
-              <height>${video_height}</height>
-              <format>RGB_INT8</format>
-            </image>
-            <clip>
-              <near>${min_depth}</near>
-              <far>${max_depth}</far>
-            </clip>
-            <noise>
-              <type>gaussian</type>
-              <mean>0.0</mean>
-              <stddev>0.05</stddev>
-            </noise>
-          </camera>
-          <always_on>1</always_on>
-          <update_rate>${rate}</update_rate>
-          <visualize>false</visualize>
-          <plugin name="${node_name}" filename="libgazebo_ros_camera.so">
-            <ros>
-              <namespace>${node_namespace}/${node_name}</namespace>
-            </ros>
-            <camera_name>${node_name}</camera_name>
-            <frame_name>${optical_frame}</frame_name>
-          </plugin>
-        </sensor>
-      </gazebo>
-    </xacro:if>
-    <xacro:if value="${gazebo_ignition}">
-      <gazebo reference="${reference_frame}">
-        <sensor name="${node_name}" type="camera">
-            <camera name="${node_name}">
+    <gazebo reference="${frame_prefix}optical_frame_link">
+      <sensor name="${frame_prefix}sensor" type="camera">
+          <camera name="${frame_prefix}camera">
+            <camera_info_topic>color/camera_info_${id}</camera_info_topic>
             <horizontal_fov>${radians(horizontal_fov)}</horizontal_fov>
             <vertical_fov>${radians(float(vertical_fov))}</vertical_fov>
@@ -71,14 +32,12 @@
                 <stddev>0.05</stddev>
             </noise>
-            </camera>
-            <always_on>1</always_on>
-            <update_rate>${rate}</update_rate>
-            <visualize>false</visualize>
-            <topic>${node_namespace}/${node_name}/color/image_raw</topic>
-            <gz_frame_id>${optical_frame}</gz_frame_id>
-            <camera_info_topic>${node_namespace}/${node_name}/color/camera_info</camera_info_topic>
-        </sensor>
-      </gazebo>
-    </xacro:if>
+          </camera>
+          <always_on>1</always_on>
+          <update_rate>${rate}</update_rate>
+          <visualize>true</visualize>
+          <topic>color/image_raw_${id}</topic>
+          <gz_frame_id>${name_prefix}${id}/${frame_prefix}optical_frame_link</gz_frame_id>
+      </sensor>
+    </gazebo>
   </xacro:macro>
 </robot>

File: urdf/gps/gps.urdf.xacro (robot description, xacro)
@@ -2,15 +2,6 @@
 <robot name="sensor_gps" xmlns:xacro="http://wiki.ros.org/xacro">
   <xacro:include filename="$(find robotnik_sensors)/urdf/gps/gps_plugin.urdf.xacro" />
-	<xacro:macro name="sensor_gps"
-               params="frame_prefix
-                       parent
-                       *origin
-                       gazebo_classic:=false
-                       gazebo_ignition:=false
-                       node_name:=gps
-                       node_namespace:=${None}
-                       topic_prefix:=~/
-                       update_rate:=5.0">
-	  <joint name="${frame_prefix}joint" type="fixed">
+	<xacro:macro name="sensor_gps" params="id frame_prefix name_prefix parent *origin">
+	  <joint name="${frame_prefix}base_joint" type="fixed">
 	    <xacro:insert_block name="origin"/>
 	    <parent link="${parent}"/>
@@ -39,4 +30,10 @@
 	    </collision>
 	  </link>
+    <joint name="${frame_prefix}joint" type="fixed">
+        <parent link="${frame_prefix}base_link"/>
+        <child link="${frame_prefix}link"/>
+        <origin xyz="0.00 0 0.0" rpy="0 0 0"/>
+    </joint>
+    <link name="${frame_prefix}link" />
 	  <gazebo reference="${frame_prefix}base_link">
 	    <material>Gazebo/White</material>
@@ -44,11 +41,7 @@
 	  </gazebo>
     <xacro:gps_plugin
-      node_namespace="${node_namespace}"
-      node_name="${node_name}"
-      gazebo_classic="${gazebo_classic}"
-      gazebo_ignition="${gazebo_ignition}"
-      topic_prefix="${topic_prefix}_gps"
-      frame_link="${frame_prefix}base_link"
-      rate="${update_rate}"
+      frame_prefix="${frame_prefix}"
+      name_prefix="${name_prefix}"
+      rate="5.0"
     >
     </xacro:gps_plugin>

File: urdf/gps/gps_plugin.urdf.xacro (robot description, xacro)
@@ -2,18 +2,11 @@
 <robot name="gps_plugin" xmlns:xacro="http://wiki.ros.org/xacro">
   <xacro:macro name="gps_plugin" params="
-            node_namespace
-            node_name
-            frame_link
-            topic_prefix
-            gazebo_classic
-            gazebo_ignition
+            frame_prefix
+            name_prefix
             rate
             ">
-    <xacro:if value="${gazebo_classic}">
-        <gazebo reference="${frame_link}">
-            <sensor type="gps" name="${node_name}">
-            <always_on>true</always_on>
-            <update_rate>${rate}</update_rate>
-            <gps>
+    <gazebo reference="${frame_prefix}link">
+        <sensor name="${frame_prefix}sensor" type="navsat">
+            <!-- <navsat>
                 <position_sensing>
                 <horizontal>
@@ -44,56 +37,11 @@
                 </vertical>
                 </vertical_sensing>
-            </gps>
-            <plugin name="${node_name}" filename="libgazebo_ros_gps_sensor.so">
-                <ros>
-                <namespace>${node_namespace}</namespace>
-                <remapping>~/out:=${topic_prefix}fix</remapping>
-                <remapping>~/vel:=${topic_prefix}vel</remapping>
-                </ros>
-            </plugin>
-            </sensor>
-        </gazebo>
-    </xacro:if>
-    <xacro:if value="${gazebo_ignition}">
-        <gazebo reference="${frame_link}">
-            <sensor name="${node_name}" type="navsat">
-                <navsat>
-                    <position_sensing>
-                    <horizontal>
-                        <noise type="gaussian">
-                        <mean>0.0</mean>
-                        <stddev>0.1</stddev>
-                        </noise>
-                    </horizontal>
-                    <vertical>
-                        <noise type="gaussian">
-                        <mean>0.0</mean>
-                        <stddev>0.1</stddev>
-                        </noise>
-                    </vertical>
-                    </position_sensing>
-                    <vertical_sensing>
-                    <horizontal>
-                        <noise type="gaussian">
-                        <mean>0.0</mean>
-                        <stddev>0.1</stddev>
-                        </noise>
-                    </horizontal>
-                    <vertical>
-                        <noise type="gaussian">
-                        <mean>0.0</mean>
-                        <stddev>0.1</stddev>
-                        </noise>
-                    </vertical>
-                    </vertical_sensing>
-                </navsat>
-                <always_on>1</always_on>
-                <update_rate>${rate}</update_rate>
-                <topic>${node_namespace}/${node_name}/data</topic>
-                <gz_frame_id>${frame_link}</gz_frame_id>
-                <plugin filename="ignition-gazebo-navsat-system" name="ignition::gazebo::systems::NavSat"/>
-            </sensor>
-        </gazebo>
-    </xacro:if>
+            </navsat> -->
+            <always_on>1</always_on>
+            <update_rate>${rate}</update_rate>
+            <topic>navsat_data_${id}</topic>
+            <gz_frame_id>${name_prefix}${id}/${frame_prefix}link</gz_frame_id>
+        </sensor>
+    </gazebo>
   </xacro:macro>
 </robot>

File: urdf/imu/imu_plugin.urdf.xacro (robot description, xacro)
@@ -3,4 +3,5 @@
   <xacro:macro name="imu_plugin" params="
             frame_prefix
+            name_prefix
             rate
             ">

File: urdf/imu/pixhawk.urdf.xacro (robot description, xacro)
@@ -39,4 +39,5 @@
     <xacro:imu_plugin
       frame_prefix="${frame_prefix}"
+      name_prefix="${name_prefix}"
       rate="200.0"
     >

Commit message: Change cam struct

File: urdf/camera/axis_m5013.urdf.xacro (robot description, xacro)
@@ -38,12 +38,12 @@
       </collision>
     </link>
-    <joint name="${frame_prefix}pan_joint" type="fixed">
-      <!-- <axis xyz="1 0 0"/> -->
+    <joint name="${frame_prefix}pan_joint" type="revolute">
+      <axis xyz="1 0 0"/>
       <origin xyz="0.04 0.0 0.0" rpy="0 0 0"/>
       <!-- check the displacement -->
       <parent link="${frame_prefix}base_link"/>
       <child link="${frame_prefix}pan_link"/>
-      <!-- <limit effort="${ptz_joint_effort_limit}" velocity="${ptz_joint_velocity_limit}" lower="-3.1416" upper="3.1416"/>
-      <joint_properties damping="${ptz_joint_damping}" friction="{ptz_joint_friction}"/> -->
+      <limit effort="${ptz_joint_effort_limit}" velocity="${ptz_joint_velocity_limit}" lower="-3.1416" upper="3.1416"/>
+      <joint_properties damping="${ptz_joint_damping}" friction="{ptz_joint_friction}"/>
     </joint>
     <link name="${frame_prefix}pan_link">
@@ -54,11 +54,11 @@
       </inertial>
     </link>
-    <joint name="${frame_prefix}tilt_joint" type="fixed">
-      <!-- <axis xyz="0 -1 0"/> -->
+    <joint name="${frame_prefix}tilt_joint" type="revolute">
+      <axis xyz="0 -1 0"/>
       <origin xyz="0.0 0.0 0.0" rpy="0 ${-PI/2} 0"/>
       <parent link="${frame_prefix}pan_link"/>
       <child link="${frame_prefix}tilt_link"/>
-      <!-- <limit effort="${ptz_joint_effort_limit}" velocity="${ptz_joint_velocity_limit}" lower="-1.5708" upper="1.5708"/>
-      <joint_properties damping="${ptz_joint_damping}" friction="{ptz_joint_friction}"/> -->
+      <limit effort="${ptz_joint_effort_limit}" velocity="${ptz_joint_velocity_limit}" lower="-1.5708" upper="1.5708"/>
+      <joint_properties damping="${ptz_joint_damping}" friction="{ptz_joint_friction}"/>
     </joint>
     <link name="${frame_prefix}tilt_link">
@@ -83,5 +83,5 @@
     <!-- Optical frame -->
     <joint name="${frame_prefix}optical_joint" type="fixed">
-      <origin xyz="0 0 0" rpy="${-PI/2} 0 ${-PI/2}"/>
+      <origin xyz="0 0 0" rpy="0 0 ${-PI/2}"/>
       <parent link="${frame_prefix}frame_link"/>
       <child link="${frame_prefix}optical_frame_link"/>

Commit message: Rm material tags

File: urdf/camera/axis_m5013.urdf.xacro (robot description, xacro)
@@ -24,7 +24,7 @@
         <origin xyz="0 0 0" rpy="0 ${PI/2} 0"/>
         <!-- to center the axis model -->
-        <material name="axis_color">
+        <!-- <material name="axis_color">
           <color rgba="0.1 0.1 0.1 1"/>
-        </material>
+        </material> -->
         <geometry>
           <mesh filename="package://robotnik_sensors/meshes/axis_m5013.dae" scale="1.0 1.0 1.0"/>

File: urdf/gps/gps.urdf.xacro (robot description, xacro)
@@ -16,7 +16,7 @@
 	    <visual>
 	      <origin rpy="0 0 0" xyz="0 0 0"/>
-	      <material name="gps_color">
+	      <!-- <material name="gps_color">
            <color rgba="1 1 1 1"/>
-        </material>
+        </material> -->
 	      <geometry>
 	        <mesh filename="package://robotnik_sensors/meshes/gps/antenna_3GO16.stl"/>

File: urdf/imu/pixhawk.urdf.xacro (robot description, xacro)
@@ -16,7 +16,7 @@
       <visual>
         <origin rpy="0 0 0" xyz="0 0 0"/>
-        <material name="pixhawk_imu_color">
+        <!-- <material name="pixhawk_imu_color">
           <color rgba="1 0 0 1"/>
-        </material>
+        </material> -->
         <geometry>
           <box size="0.05 0.0815 0.0155"/>

Commit message: Add depth camera

File: urdf/camera/axis_m5013.urdf.xacro (robot description, xacro)
@@ -83,5 +83,5 @@
     <!-- Optical frame -->
     <joint name="${frame_prefix}optical_joint" type="fixed">
-      <origin xyz="0 0 0" rpy="0 0 ${-PI/2}"/>
+      <origin xyz="0 0 0" rpy="0 ${75*PI/180} 0"/>
       <parent link="${frame_prefix}frame_link"/>
       <child link="${frame_prefix}optical_frame_link"/>

File: urdf/depth/azure_kinect.urdf.xacro (robot description, xacro)
@@ -3,15 +3,5 @@
   <xacro:include filename="$(find robotnik_sensors)/urdf/depth/depth_camera_plugin.urdf.xacro" />
   <xacro:macro name="sensor_azure_kinect"
-               params="frame_prefix
-                       parent
-                       *origin
-                       gazebo_classic:=false
-                       gazebo_ignition:=false
-                       node_namespace:=${None}
-                       node_name:=azure_kinect
-                       topic_prefix:=~/">
-    <xacro:if value="${node_namespace == None}">
-      <xacro:property name="node_namespace" value="${node_name}"/>
-    </xacro:if>
+               params="id frame_prefix name_prefix parent *origin">
     <joint name="${frame_prefix}joint" type="fixed">
     	<xacro:insert_block name="origin" />
@@ -74,5 +64,5 @@
     <link name="${frame_prefix}depth_frame"/>
     <joint name="${frame_prefix}depth_optical_joint" type="fixed">
-      <origin xyz="0 0 0" rpy="${-PI/2} 0 ${-PI/2}" />
+      <origin xyz="0.1 0 0" rpy="${-PI/2} 0 ${-PI/2}" />
       <parent link="${frame_prefix}depth_frame" />
       <child link="${frame_prefix}depth_optical_frame" />
@@ -90,11 +80,6 @@
     <!-- RGBD sensor for simulation, same as Kinect -->
     <xacro:depth_camera_plugin
-      node_namespace="${node_namespace}"
-      node_name="${node_name}"
-      topic_prefix="${topic_prefix}"
-      gazebo_classic="${gazebo_classic}"
-      gazebo_ignition="${gazebo_ignition}"
-      optical_frame="${frame_prefix}color_optical_frame"
-      reference_frame="${frame_prefix}color_frame"
+      frame_prefix="${frame_prefix}"
+      name_prefix="${name_prefix}"
       horizontal_fov="60"
       vertical_fov="45"

File: urdf/depth/depth_camera_plugin.urdf.xacro (robot description, xacro)
@@ -2,11 +2,6 @@
 <robot name="depth_camera_plugin" xmlns:xacro="http://wiki.ros.org/xacro">
   <xacro:macro name="depth_camera_plugin" params="
-            node_namespace
-            node_name
-            topic_prefix
-            gazebo_classic
-            gazebo_ignition
-            optical_frame
-            reference_frame
+            frame_prefix
+            name_prefix
             horizontal_fov
             vertical_fov
@@ -17,78 +12,31 @@
             rate
             ">
-    <xacro:if value="${gazebo_classic}">
-      <gazebo reference="${reference_frame}">
-        <sensor name="${node_name}" type="depth">
-          <pose>0.0 0.0 0.0 0.0 0.0 0.0</pose>
-          <visualize>false</visualize>
-          <update_rate>${rate}</update_rate>
-          <camera>
-            <horizontal_fov>${radians(float(horizontal_fov))}</horizontal_fov>
-            <vertical_fov>${radians(float(vertical_fov))}</vertical_fov>
-            <image>
-              <width>${video_width}</width>
-              <height>${video_height}</height>
-              <format>B8G8R8</format>
-            </image>
-            <clip>
-              <near>${min_depth}</near>
-              <far>${max_depth}</far>
-            </clip>
-            <noise>
-              <type>gaussian</type>
-              <mean>0.0</mean>
-              <stddev>0.007</stddev>
-            </noise>
-          </camera>
-          <plugin name="${node_name}" filename="libgazebo_ros_camera.so">
-            <ros>
-              <namespace>${node_namespace}</namespace>
-              <remapping>~/image_raw:=${topic_prefix}rgb/image_raw_color</remapping>
-              <remapping>~/camera_info:=${topic_prefix}rgb/camera_info</remapping>
-              <remapping>~/points:=${topic_prefix}point_cloud/cloud_registered</remapping>
-              <remapping>~/depth/camera_info:=${topic_prefix}depth/camera_info</remapping>
-              <remapping>~/depth/image_raw:=${topic_prefix}depth/depth_registered</remapping>
-            </ros>
-            <camera_name>${node_name}</camera_name>
-            <frame_name>${optical_frame}</frame_name>
-            <min_depth>${min_depth}</min_depth>
-            <max_depth>${max_depth}</max_depth>
-          </plugin>
-        </sensor>
-      </gazebo>
-    </xacro:if>
-    <xacro:if value="${gazebo_ignition}">
-      <gazebo reference="${reference_frame}">
-        <sensor name="${node_name}" type="depth">
-          <camera name="${node_name}">
-            <camera_info_topic>${node_name}/depth/camera_info</camera_info_topic>
-            <horizontal_fov>${radians(float(horizontal_fov))}</horizontal_fov>
-            <vertical_fov>${radians(float(vertical_fov))}</vertical_fov>
-            <image>
-              <width>${video_width}</width>
-              <height>${video_height}</height>
-              <format>B8G8R8</format>
-            </image>
-            <clip>
-              <near>${min_depth}</near>
-              <far>${max_depth}</far>
-            </clip>
-            <noise>
-              <type>gaussian</type>
-              <mean>0.0</mean>
-              <stddev>0.100</stddev>
-            </noise>
-          </camera>
-          <always_on>1</always_on>
-          <update_rate>30</update_rate>
-          <visualize>false</visualize>
-          <camera_info_topic>${node_namespace}/${node_name}/depth/camera_info</camera_info_topic>
-          <topic>${node_namespace}/${node_name}/depth/image_raw</topic>
-          <gz_frame_id>${optical_frame}</gz_frame_id>
-          <min_depth>${min_depth}</min_depth>
-          <max_depth>${max_depth}</max_depth>
-        </sensor>
-      </gazebo>
-    </xacro:if>
+    <gazebo reference="${frame_prefix}depth_optical_frame">
+      <sensor name="${frame_prefix}sensor" type="rgbd_camera">
+        <camera name="$frame_prefix}camera">
+          <horizontal_fov>${radians(float(horizontal_fov))}</horizontal_fov>
+          <vertical_fov>${radians(float(vertical_fov))}</vertical_fov>
+          <image>
+            <width>${video_width}</width>
+            <height>${video_height}</height>
+            <format>B8G8R8</format>
+          </image>
+          <clip>
+            <near>${min_depth}</near>
+            <far>${max_depth}</far>
+          </clip>
+          <noise>
+            <type>gaussian</type>
+            <mean>0.0</mean>
+            <stddev>0.100</stddev>
+          </noise>
+        </camera>
+        <always_on>1</always_on>
+        <update_rate>30</update_rate>
+        <visualize>true</visualize>
+        <topic>depth/image_raw_${id}</topic>
+        <gz_frame_id> ${name_prefix}${id}/${frame_prefix}depth_optical_frame </gz_frame_id>
+      </sensor>
+    </gazebo>
   </xacro:macro>
 </robot>
